File: hardware/xbee_module/zigbee_iNEMO.brd (EAGLE design)
At the start: 50.3 x 56.2 mm, 42 parts, among them J2 6_PIN_SERIAL_CABLEPTH, Q1 2.5A/30V/105mΩ, U1 TS3A4751, U10 HTS221TRHLGA-6L_2X2_STM-M, U3 XBEE3_Micro, U4 LTC3106EUDC#TRPBF, U9 ISM330DHCXTR

Commit message: Uploading gerber files
Parts:
- moved J2 78.9 mm to (11.6, 54.4), turned to 270 degrees
- moved R3 67.0 mm to (16.7, 45.4), turned to 90 degrees
- moved R12 44.6 mm to (14.7, 20.7)
- moved RESET1 38.0 mm to (10.7, 16.8), turned to 270 degrees
- moved S1 33.5 mm to (14.6, 16.8), turned to 90 degrees
- moved U3 24.0 mm to (9.63, 29.2), turned to 90 degrees
- moved C15 17.7 mm to (10.9, 20.7)
- moved C13 10.5 mm to (26.9, 32.6)
- moved U1 10.5 mm to (29.6, 29.7)
- moved R4 10.5 mm to (31.5, 23.4)
- moved R1 10.5 mm to (36.2, 29.9)
- moved C16 10.4 mm to (26.8, 26.8)
- moved R6 10.2 mm to (36.1, 28.3)
- moved D1 2.35 mm to (16.7, 48.9), turned to 90 degrees
Connections:
- removed net 3.3V: C12.1, J1.2, R8.2, R9.2
- removed net SCL_1.8V: U9.3
- removed net SDA_1.8V: U9.2
- net SCL_AUX: now also U9.3
- net SDA: now also U1.3; no longer U1.9
- net SDA_AUX: now also U9.2
- net SDA_OUT: now also U1.4; no longer U1.8
- net VCC_1: now also C12.1, J1.2, R8.2, R9.2
Routing:
- net VDD: track 154.9 -> 89.1 mm, vias 9 -> 6
- net DOUT: track 0.00 -> 48.1 mm, vias 0 -> 2
- net DIN: track 0.00 -> 41.8 mm, vias 0 -> 2
- net !SLEEP_RQ: track 0.00 -> 41.7 mm, vias 0 -> 1
- net RESET: track 36.3 -> 8.01 mm
- net 3.3V: track 25.3 -> 0.00 mm, vias 2 -> 0
- net VCC_1: track 88.0 -> 107.7 mm, vias 9 -> 8
- net ASSOC: track 0.00 -> 17.9 mm, vias 0 -> 2
- net SDA_1.8V: track 16.9 -> 0.00 mm, vias 2 -> 0
- net SDA_OUT: track 46.4 -> 62.5 mm
- net SCL: track 15.2 -> 31.2 mm
- net SENSOR_EN1: track 22.3 -> 38.3 mm
- net CTS: track 0.00 -> 15.9 mm, vias 0 -> 2
- net SCL_1.8V: track 13.3 -> 0.00 mm, vias 2 -> 0
- net SCL_OUT: track 49.6 -> 38.2 mm
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