File: hardware/xbee_module/zigbee_iNEMO.sch (EAGLE design)
At the start: 42 parts, among them J2 6_PIN_SERIAL_CABLEPTH, Q1 2.5A/30V/105mΩ, U1 TS3A4751, U10 HTS221TRHLGA-6L_2X2_STM-M, U3 XBEE3_Micro, U4 LTC3106EUDC#TRPBF, U9 ISM330DHCXTR

Commit message: Uploading gerber files
Connections:
- removed net 3.3V: C12.1, J1.2, R8.2, R9.2
- removed net SCL_1.8V: U9.SCX
- removed net SDA_1.8V: U9.SDX
- net SCL_AUX: now also U9.SCX
- net SDA: now also U1.NO2; no longer U1.COM3
- net SDA_AUX: now also U9.SDX
- net SDA_OUT: now also U1.COM2; no longer U1.NO3
- net VCC_1: now also C12.1, J1.2, R8.2, R9.2
Changed lines of the file:
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@@
 <?xml version="1.0" encoding="utf-8"?>
 <!DOCTYPE eagle SYSTEM "eagle.dtd">
-<eagle version="9.6.2">
+<eagle version="9.6.0">
 <drawing>
 <settings>
@@
 <part name="R8" library="SparkFun-Resistors" library_urn="urn:adsk.eagle:library:532" deviceset="4.7KOHM" device="-0603-1/10W-1%" package3d_urn="urn:adsk.eagle:package:39650/1" value="4.7k"/>
 <part name="R9" library="SparkFun-Resistors" library_urn="urn:adsk.eagle:library:532" deviceset="4.7KOHM" device="-0603-1/10W-1%" package3d_urn="urn:adsk.eagle:package:39650/1" value="4.7k"/>
-<part name="SUPPLY6" library="SparkFun-PowerSymbols" library_urn="urn:adsk.eagle:library:530" deviceset="3.3V" device=""/>
-<part name="SUPPLY10" library="SparkFun-PowerSymbols" library_urn="urn:adsk.eagle:library:530" deviceset="3.3V" device=""/>
 <part name="U3" library="starview_mini_v7" deviceset="XBEE3_THING_PLUS_SPARKFUN-RF_XBEE3" device="" value="XBEE3_Micro"/>
 <part name="GND23" library="supply1" library_urn="urn:adsk.eagle:library:371" deviceset="GND" device=""/>
@@
 <part name="SUPPLY8" library="SparkFun-PowerSymbols" library_urn="urn:adsk.eagle:library:530" deviceset="VDD" device=""/>
 <part name="SUPPLY1" library="SparkFun-PowerSymbols" deviceset="VCC_1" device=""/>
+<part name="SUPPLY7" library="SparkFun-PowerSymbols" deviceset="VCC_1" device=""/>
+<part name="SUPPLY6" library="SparkFun-PowerSymbols" deviceset="VCC_1" device=""/>
 </parts>
 <sheets>
@@
 <attribute name="VALUE" x="237.236" y="48.514" size="1.016" layer="96" font="vector" ratio="20" rot="MR180" align="top-center"/>
 </instance>
-<instance part="SUPPLY6" gate="G$1" x="251.206" y="59.944" smashed="yes">
-<attribute name="VALUE" x="251.206" y="62.738" size="1.016" layer="96" font="vector" ratio="20" align="bottom-center"/>
-</instance>
-<instance part="SUPPLY10" gate="G$1" x="159.004" y="81.026" smashed="yes">
-<attribute name="VALUE" x="159.004" y="83.82" size="1.016" layer="96" font="vector" ratio="20" align="bottom-center"/>
-</instance>
 <instance part="SUPPLY4" gate="VDD" x="17.78" y="86.36" smashed="yes">
 <attribute name="VALUE" x="17.78" y="89.154" size="1.016" layer="96" font="vector" ratio="20" align="bottom-center"/>
@@
 <instance part="SUPPLY1" gate="G$2" x="25.146" y="86.106" smashed="yes">
 <attribute name="VALUE" x="27.686" y="86.36" size="1.016" layer="96" font="vector" ratio="20" align="bottom-center"/>
+</instance>
+<instance part="SUPPLY7" gate="G$2" x="158.75" y="75.692" smashed="yes">
+<attribute name="VALUE" x="161.29" y="75.946" size="1.016" layer="96" font="vector" ratio="20" align="bottom-center"/>
+</instance>
+<instance part="SUPPLY6" gate="G$2" x="251.206" y="59.944" smashed="yes">
+<attribute name="VALUE" x="253.746" y="60.198" size="1.016" layer="96" font="vector" ratio="20" align="bottom-center"/>
 </instance>
 </instances>
@@
 <pinref part="SUPPLY1" gate="G$2" pin="VCC_1"/>
 </segment>
+<segment>
+<pinref part="J1" gate="G$1" pin="2"/>
+<wire x1="137.16" y1="55.88" x2="149.352" y2="55.88" width="0.1524" layer="91"/>
+<wire x1="149.352" y1="55.88" x2="149.352" y2="65.786" width="0.1524" layer="91"/>
+<pinref part="C12" gate="G$1" pin="1"/>
+<wire x1="159.004" y1="61.468" x2="159.004" y2="65.786" width="0.1524" layer="91"/>
+<wire x1="159.004" y1="65.786" x2="158.75" y2="65.786" width="0.1524" layer="91"/>
+<pinref part="SUPPLY7" gate="G$2" pin="VCC_1"/>
+<wire x1="158.75" y1="65.786" x2="149.352" y2="65.786" width="0.1524" layer="91"/>
+<wire x1="158.75" y1="65.786" x2="158.75" y2="75.692" width="0.1524" layer="91"/>
+<junction x="158.75" y="65.786"/>
+</segment>
+<segment>
+<pinref part="R8" gate="G$1" pin="2"/>
+<wire x1="246.38" y1="53.34" x2="251.206" y2="53.34" width="0.1524" layer="91"/>
+<wire x1="251.206" y1="53.34" x2="251.206" y2="59.944" width="0.1524" layer="91"/>
+<pinref part="R9" gate="G$1" pin="2"/>
+<wire x1="246.38" y1="48.26" x2="251.206" y2="48.26" width="0.1524" layer="91"/>
+<wire x1="251.206" y1="48.26" x2="251.206" y2="53.34" width="0.1524" layer="91"/>
+<junction x="251.206" y="53.34"/>
+<pinref part="SUPPLY6" gate="G$2" pin="VCC_1"/>
+</segment>
 </net>
 <net name="SENSOR_EN1" class="0">
@@
 </segment>
 <segment>
-<pinref part="U1" gate="G$1" pin="NO3"/>
-<wire x1="58.42" y1="53.34" x2="63.5" y2="53.34" width="0.1524" layer="91"/>
-<label x="63.5" y="53.34" size="1.016" layer="95" font="vector" ratio="20" xref="yes"/>
-</segment>
-</net>
-<net name="SDA" class="0">
-<segment>
-<pinref part="U1" gate="G$1" pin="COM3"/>
-<wire x1="58.42" y1="55.88" x2="63.5" y2="55.88" width="0.1524" layer="91"/>
-<label x="63.5" y="55.88" size="1.016" layer="95" font="vector" ratio="20" xref="yes"/>
+<pinref part="U1" gate="G$1" pin="COM2"/>
+<wire x1="27.94" y1="60.96" x2="22.86" y2="60.96" width="0.1524" layer="91"/>
+<label x="22.86" y="60.96" size="1.016" layer="95" font="vector" ratio="20" rot="R180" xref="yes"/>
 </segment>
 </net>
@@
 <label x="226.06" y="48.26" size="1.016" layer="95" font="vector" ratio="20" rot="R180" xref="yes"/>
 </segment>
+<segment>
+<pinref part="U9" gate="A" pin="SDX"/>
+<wire x1="160.02" y1="124.46" x2="154.94" y2="124.46" width="0.1524" layer="91"/>
+<label x="154.94" y="124.46" size="1.016" layer="95" font="vector" ratio="20" rot="R180" xref="yes"/>
+</segment>
 </net>
 <net name="SCL_AUX" class="0">
@@
 <label x="226.06" y="53.34" size="1.016" layer="95" font="vector" ratio="20" rot="R180" xref="yes"/>
 </segment>
-</net>
-<net name="3.3V" class="0">
-<segment>
-<pinref part="R8" gate="G$1" pin="2"/>
-<wire x1="246.38" y1="53.34" x2="251.206" y2="53.34" width="0.1524" layer="91"/>
-<wire x1="251.206" y1="53.34" x2="251.206" y2="59.944" width="0.1524" layer="91"/>
-<pinref part="R9" gate="G$1" pin="2"/>
-<wire x1="246.38" y1="48.26" x2="251.206" y2="48.26" width="0.1524" layer="91"/>
-<wire x1="251.206" y1="48.26" x2="251.206" y2="53.34" width="0.1524" layer="91"/>
-<junction x="251.206" y="53.34"/>
-<pinref part="SUPPLY6" gate="G$1" pin="3.3V"/>
-</segment>
-<segment>
-<pinref part="J1" gate="G$1" pin="2"/>
-<wire x1="137.16" y1="55.88" x2="149.352" y2="55.88" width="0.1524" layer="91"/>
-<wire x1="149.352" y1="55.88" x2="149.352" y2="65.786" width="0.1524" layer="91"/>
-<pinref part="C12" gate="G$1" pin="1"/>
-<wire x1="159.004" y1="61.468" x2="159.004" y2="65.786" width="0.1524" layer="91"/>
-<wire x1="159.004" y1="65.786" x2="149.352" y2="65.786" width="0.1524" layer="91"/>
-<wire x1="159.004" y1="81.026" x2="159.004" y2="65.786" width="0.1524" layer="91"/>
-<junction x="159.004" y="65.786"/>
-<pinref part="SUPPLY10" gate="G$1" pin="3.3V"/>
-</segment>
-</net>
-<net name="SDA_1.8V" class="0">
-<segment>
-<pinref part="U9" gate="A" pin="SDX"/>
-<wire x1="160.02" y1="124.46" x2="154.94" y2="124.46" width="0.1524" layer="91"/>
-<label x="154.94" y="124.46" size="1.016" layer="95" font="vector" ratio="20" rot="R180" xref="yes"/>
-</segment>
-</net>
-<net name="SCL_1.8V" class="0">
 <segment>
 <pinref part="U9" gate="A" pin="SCX"/>
@@
 </segment>
 </net>
+<net name="SDA" class="0">
+<segment>
+<pinref part="U1" gate="G$1" pin="NO2"/>
+<wire x1="27.94" y1="63.5" x2="22.86" y2="63.5" width="0.1524" layer="91"/>
+<label x="22.86" y="63.5" size="1.016" layer="95" font="vector" ratio="20" rot="R180" xref="yes"/>
+</segment>
+</net>
